File: hardware/drone_sim_controler.kicad_pcb (KiCad board)
At the start: 2 copper layers, 13.2 x 6.2 mm, 57 parts, among them J1 USB_C_Receptacle_USB2.0_14P, J2 PROG_PORT, J3 JTAG, SW1 SW_MEC_5E, SW2 SW_MEC_5E, U1 ESP32-S2FH2, U2 ECMF02-2AMX6, U3 TPS63031DSKR, Y1 40MHz

Commit message: compleeted first rev of board
Parts:
- added G***: LOGO, CONTROLER:hex, B.Cu at (96.8, 140.6)
- added TP15: ~, TestPoint:TestPoint_Pad_D1.0mm, F.Cu at (66.2, 132.8)
- added TP16: ~, TestPoint:TestPoint_Pad_D1.0mm, F.Cu at (83.3, 147.5)
- added TP17: ~, TestPoint:TestPoint_Pad_D1.0mm, F.Cu at (97.5, 152.3)
- added TP18: ~, TestPoint:TestPoint_Pad_D1.0mm, F.Cu at (114.0, 146.4)
- added TP19: ~, TestPoint:TestPoint_Pad_D1.0mm, F.Cu at (114.0, 150.4)
- added TP20: ~, TestPoint:TestPoint_Pad_D1.0mm, F.Cu at (114.0, 148.4)
- added TP21: ~, TestPoint:TestPoint_Pad_D1.0mm, F.Cu at (53.6, 146.3)
- added TP22: ~, TestPoint:TestPoint_Pad_D1.0mm, F.Cu at (53.6, 150.3)
- added TP23: ~, TestPoint:TestPoint_Pad_D1.0mm, F.Cu at (53.6, 148.3)
- added TP24: ~, TestPoint:TestPoint_Pad_D1.0mm, F.Cu at (79.9, 132.1)
- added TP25: ~, TestPoint:TestPoint_Pad_D1.0mm, F.Cu at (79.9, 134.1)
- added TP26: ~, TestPoint:TestPoint_Pad_D1.0mm, F.Cu at (79.9, 136.1)
- Y1: value 40MHz -> 40 MHz
- moved JS2 139.2 mm to (126.7, 148.4)
- moved JS1 132.1 mm to (66.7, 148.4)
- moved C2 120.1 mm to (103.3, 139.3)
- moved R10 118.5 mm to (119.8, 137.6)
- moved R1 117.4 mm to (118.9, 132.0), turned to 90 degrees
- moved R12 116.4 mm to (97.0, 150.2)
- moved C11 114.7 mm to (103.3, 137.8)
- moved C9 114.3 mm to (88.2, 138.2), turned to 180 degrees
- moved R8 113.6 mm to (88.2, 139.7), turned to 180 degrees
- moved TP11 112.8 mm to (83.3, 151.5)
- moved R11 111.0 mm to (83.3, 145.6)
- moved C1 110.9 mm to (102.4, 126.9), turned to 90 degrees
- moved C3 109.4 mm to (88.2, 136.7), turned to 180 degrees
- moved SW1 109.3 mm to (86.7, 145.6)
- moved TP12 107.8 mm to (83.3, 149.5)
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Connections:
- D2 pad 1: Net-(D2-BA) -> Net-(D2-GA)
- D2 pad 2: GND -> Net-(D2-RA)
- D2 pad 3: Net-(D2-GA) -> Net-(D2-BA)
- D2 pad 4: Net-(D2-RA) -> GND
- JS1 pad B1A: RS_SW -> LS_SW
- JS1 pad H2: RS_Y -> LS_Y
- JS1 pad V2: RS_X -> LS_X
- JS2 pad B1A: LS_SW -> RS_SW
- JS2 pad H2: LS_Y -> RS_Y
- JS2 pad V2: LS_X -> RS_X
- R10 pad 2: LS_SW -> RS_SW
- R9 pad 2: RS_SW -> LS_SW
- TP11 pad 1: Net-(U1-GPIO13) -> Net-(U1-GPIO8)
- TP12 pad 1: Net-(U1-GPIO12) -> Net-(U1-GPIO7)
- U1 pad 12: BTN_1 -> Net-(U1-GPIO7)
- U1 pad 13: BTN_2 -> Net-(U1-GPIO8)
- U1 pad 17: Net-(U1-GPIO12) -> BTN_1
- U1 pad 18: Net-(U1-GPIO13) -> BTN_2
- Y1 pad 2: Net-(U1-XTAL_N) -> GND
- Y1 pad 3: (no net) -> Net-(U1-XTAL_N)
- Y1 pad 4: (no net) -> GND
Routing:
- net GNDS: track 0.00 -> 97.3 mm
- net USB_N: track 0.00 -> 68.5 mm
- net USB_P: track 0.00 -> 68.5 mm
- net RS_Y: track 0.00 -> 66.8 mm, vias 0 -> 1
- net +3V3: track 0.00 -> 63.6 mm, vias 0 -> 15
- net LS_Y: track 0.00 -> 54.8 mm, vias 0 -> 1
- net GND: track 0.00 -> 48.9 mm, vias 0 -> 25
- net LS_X: track 0.00 -> 48.2 mm, vias 0 -> 1
- net RS_SW: track 0.00 -> 45.2 mm, vias 0 -> 1
- net LS_SW: track 0.00 -> 45.0 mm, vias 0 -> 1
- net MTDI: track 0.00 -> 40.8 mm, vias 0 -> 1
- net MTMS: track 0.00 -> 39.8 mm, vias 0 -> 1
- net MTCK: track 0.00 -> 38.0 mm, vias 0 -> 1
- net RS_X: track 0.00 -> 37.6 mm, vias 0 -> 1
- net RST: track 0.00 -> 36.0 mm, vias 0 -> 1
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- added copper zone on In2.Cu, net +3V3
- added copper zone on F.Cu, net GND
- added copper zone on In1.Cu, net GND
Other:
- board size 13.2 x 6.2 mm -> 100 x 50 mm
- copper layers 2 -> 4
- board text added: "3V3"
- board text added: "GND"
- board text added: "IO0"
- board text added: "JTAG"
- board text added: "MTCK"
- board text added: "MTDI"
- board text added: "MTDO"
- board text added: "MTMS"
- board text added: "PROG"
- board text added: "RST"
- board text added: "RX"
- board text added: "TX"
