File: hardware/drone_sim_controler.kicad_sch (KiCad schematic)
At the start: 57 parts, among them J1 USB_C_Receptacle_USB2.0_14P, J2 PROG_PORT, J3 JTAG, SW1 SW_MEC_5E, SW2 SW_MEC_5E, U1 ESP32-S2FH2, U2 ECMF02-2AMX6, U3 TPS63031DSKR, Y1 40MHz

Commit message: compleeted first rev of board
Parts:
- removed Y1: 40MHz, CONTROLER:cx3225sa_e, symbol Device:Crystal
- added TP15, TP16, TP17, TP18, TP19, TP20, TP21, TP22, TP23, TP24, TP25, TP26: ~, TestPoint:TestPoint_Pad_D1.0mm, symbol Connector:TestPoint
- added Y1: 40 MHz, CONTROLER:cx3225sa_e, symbol Device:Crystal_GND23
Connections:
- net BTN_1: now also U1.17 (GPIO12), TP16.1; no longer U1.12 (GPIO7)
- net BTN_2: now also U1.18 (GPIO13), TP17.1; no longer U1.13 (GPIO8)
- net GND: now also D2.4 (K), TP15.1, Y1.2, Y1.4; no longer D2.2 (K)
- net LS_SW: now also JS1.B1A (SW_COM), R9.2, TP21.1; no longer JS2.B1A (SW_COM), R10.2
- net LS_X: now also JS1.V2 (X_W), TP23.1; no longer JS2.V2 (X_W)
- net LS_Y: now also JS1.H2 (Y_W), TP22.1; no longer JS2.H2 (Y_W)
- net RS_SW: now also JS2.B1A (SW_COM), R10.2, TP18.1; no longer JS1.B1A (SW_COM), R9.2
- net RS_X: now also JS2.V2 (X_W), TP20.1; no longer JS1.V2 (X_W)
- net RS_Y: now also JS2.H2 (Y_W), TP19.1; no longer JS1.H2 (Y_W)
- net at TP12.1: now also U1.12 (GPIO7); no longer U1.17 (GPIO12)
- net at R7.2: now also D2.1 (GA), TP25.1; no longer D2.3 (GA)
- net at R8.2: now also D2.3 (BA), TP24.1; no longer D2.1 (BA)
- net at R6.2: now also D2.2 (RA), TP26.1; no longer D2.4 (RA)
- net at C15.1, U1.53 (XTAL_P): now also Y1.1
- net at C14.1, U1.52 (XTAL_N): now also Y1.3
- net at TP11.1: now also U1.13 (GPIO8); no longer U1.18 (GPIO13)
Other:
- moved on the sheet: C15, D2, JS1, R6, R7, R8, R9
